File: esprog.sch (EAGLE design)
At the start: 12 parts, among them J1 MICRO-USB-5P-340015001, U1 FT232RL-1720010P1, U2 CJ1117-3.3-1310190P1

Commit message: Final v1.0 PCB - Added PCB Design - Finished Circuit Schematic
Parts:
- added J2, J3: CONNECTOR-HEADER-8P-3460290P1, Connector:CONNECTOR-HEADER-8P-3460290P1
- added R1, R2: 1K, Discrete:R-0805
- added R3, R4: 10K, Discrete:R-0805
- added U$1: ESP8266_ESP-03, ESP8266:ESP8266_ESP-03
- C1: value 10nF -> 100nF
- C2: value 100nF -> 10nF
- C3: value 10uF -> 4.7uF; device Discrete:CAP-POLAR-AVX-B -> Discrete:CAP-0805
- C4: value 22uF -> 100nF; device Discrete:CAP-POLAR-AVX-B -> Discrete:CAP-0603
- C5: value 100nF -> 10uF; device Discrete:CAP-0603 -> Discrete:CAP-POLAR-AVX-B
- C6: value 4.7uF -> 22uF; device Discrete:CAP-0805 -> Discrete:CAP-POLAR-AVX-B
- D1: value (none) -> TX
- D2: value (none) -> RX
- L1: value (none) -> 120 OHM 500MA
- U1: value FT232RL-1720010P1 -> CJ1117-3.3-1310190P1; device IC:FT232RL-1720010P1 -> IC:CJ1117-3.3-1310190P1
- U2: value CJ1117-3.3-1310190P1 -> FT232RL-1720010P1; device IC:CJ1117-3.3-1310190P1 -> IC:FT232RL-1720010P1
Connections:
- removed net N$2: U1.TXD
- removed net N$6: J1.DP, U1.USBDP
- removed net VCC: C2.1, U1.3V3OUT, U1.VCCIO
- new net DM: J1.DM, U2.USBDM
- new net DP: J1.DP, U2.USBDP
- new net ESP_GPIO12: J2.6, U$1.GPIO12
- new net ESP_GPIO13: J2.5, U$1.GPIO13
- new net ESP_GPIO14: J2.7, U$1.GPIO14
- new net ESP_GPIO15: J2.4, R3.1, U$1.GPIO15
- new net ESP_GPIO16: U$1.GPIO16
- new net ESP_GPIO2: J2.3, U$1.GPIO2
- new net ESP_UPG: J2.2, R4.1, U$1.GPIO0, U2.CBUS4
- new net FT_RXD: J3.3, U$1.TX, U2.RXD
- new net FT_TXD: J3.4, U$1.RX, U2.TXD
- new net N$1: D1.+, R1.2
- new net N$7: D2.+, R2.2
- new net RX_LED: D2.-, U2.CBUS1
- new net TX_LED: D1.-, U2.CBUS0
- new net VCCIO: C4.1, R1.1, R2.1, U2.3V3OUT, U2.VCCIO
- new net VUSB: C2.1, J1.VCC, L1.1
- net +3V3: now also C6.+, J2.8, R4.2, U$1.CH_PD, U$1.VCC, U1.OUT; no longer C4.+, U2.OUT
- net +5V: now also C1.1, C3.1, C5.+, J3.8, U1.IN, U2.VCC; no longer C3.+, C5.1, C6.1, U1.VCC, U2.IN
- net GND: now also C3.2, C4.2, C5.-, C6.-, J2.1, J3.1, J3.2, R3.2, U$1.GND, U2.GND@1, U2.GND@2, U2.GND@A; no longer C3.-, C4.-, C5.2, C6.2, U1.GND@1, U1.GND@2, U1.GND@A
- net N$3: now also J3.7; no longer U1.RXD
- net N$4: now also J3.6; no longer J1.DM, U1.USBDM
- net N$5: now also J3.5; no longer C1.1, J1.VCC, L1.1
Other:
- moved on the sheet: C1, C2, D1, D2, L1
